Commit message: Jacobs final commit

File: jacob_arm/src/robot_description/urdf/Arm_assembly.urdf.xacro (robot description, xacro)
@@ -85,5 +85,5 @@
   <joint
     name="Joint1"
-    type="continuous">
+    type="revolute">
     <origin
       xyz="0 0 0.0637999999999999"
@@ -95,4 +95,9 @@
     <axis
       xyz="0 0 1" />
+    <limit
+        lower="-3.14"
+        upper="3.14"
+        effort="100"
+        velocity="2.0"/>
   </joint>
   <joint name="base2world" type="fixed">
@@ -141,5 +146,5 @@
   <joint
     name="Joint2"
-    type="continuous">
+    type="revolute">
     <origin
       xyz="0.0493654257105637 0.0629674380302429 0.096866312640014"
@@ -151,4 +156,9 @@
     <axis
       xyz="-0.998759127785777 0.0498016532315323 0" />
+    <limit
+        lower="-3.14"
+        upper="3.14"
+        effort="100"
+        velocity="2.0"/>
   </joint>
   <link
@@ -192,5 +202,5 @@
   <joint
     name="Joint3"
-    type="continuous">
+    type="revolute">
     <origin
       xyz="0.0150729083014778 -0.149509002764561 0.330901216092781"
@@ -202,4 +212,9 @@
     <axis
       xyz="-0.998759127785812 0.0498016532308395 0" />
+    <limit
+        lower="-3.14"
+        upper="3.14"
+        effort="100"
+        velocity="2.0"/>
   </joint>
   <link
@@ -249,5 +264,5 @@
   <joint
     name="Joint4"
-    type="continuous">
+    type="revolute">
     <origin
       xyz="-0.0336807621063758 -0.173467508873688 0.177903552627862"
@@ -259,4 +274,9 @@
     <axis
       xyz="0.998759127785812 -0.0498016532308386 0" />
+    <limit
+        lower="-3.14"
+        upper="3.14"
+        effort="100"
+        velocity="2.0"/>
   </joint>
   <link
@@ -300,5 +320,5 @@
   <joint
     name="Joint5"
-    type="continuous">
+    type="revolute">
     <origin
       xyz="0.141823796145833 -0.00707183594519112 0.0758294127267807"
@@ -310,4 +330,9 @@
     <axis
       xyz="0 0 -1" />
+    <limit
+        lower="-3.14"
+        upper="3.14"
+        effort="100"
+        velocity="2.0"/>
   </joint>
   <link
