Commit message: Integrated perception with 5dof

File: rcup_final/src/robot/urdf/merged_robot.xacro (robot description, xacro)
@@ -1188,9 +1188,9 @@
     <parent link="camera_link"/>
     <child link="camera_optical_link"/>
-    <origin xyz="0 0 0" rpy="0 1.5708 1.5708"/>
+    <origin xyz="0 0 0" rpy="-1.5707963267948966 0 -1.5707963267948966"/>
   </joint>
   <gazebo reference="camera_link">
     <sensor name="rgbd_camera" type="rgbd_camera">
-      <pose>0 0 0.07 0 0 0</pose>
+      <pose>0.0127 0 0 0 0 0</pose>
       <camera>
         <horizontal_fov>1.477</horizontal_fov>
@@ -1208,4 +1208,5 @@
       <visualize>true</visualize>
       <topic>rgbd_camera</topic>
+      <gz_frame_id>camera_optical_link</gz_frame_id>
     </sensor>
 </gazebo>
