Commit message: Added perception, integration left

File: rcup_assembly/src/piper_description/urdf/piper_arm_macro.xacro (robot description, xacro)
@@ -199,4 +199,133 @@
       <child link="${prefix}tool_0" />
     </joint>
+  <link name="camera_link">
+    <visual>
+      <origin xyz="0 0 0" rpy="0 0 0" />
+      <geometry>
+        <box size="0.025 0.09 0.025" />
+      </geometry>
+      <material name="akshit">
+        <color rgba="1 1 1 1" />
+      </material>
+    </visual>
+    <collision>
+      <origin xyz="0 0 0" rpy="0 0 0" />
+      <geometry>
+        <box size="0.06 0.03 0.03" />
+      </geometry>
+      <material name="akshit">
+        <color rgba="1 1 1 1" />
+      </material>
+    </collision>
+    <inertial>
+      <mass value="0.0000000001" />
+      <origin xyz="0 0 0" />
+      <inertia ixx="0.0000000001" ixy="0.0" ixz="0.0" iyy="0.0000000001" iyz="0.0" izz="0.0000000001" />
+    </inertial>
+  </link>
+  <!-- Horizontal Rod Link -->
+  <link name="camera_horizontal_rod">
+    <visual>
+      <origin xyz="0.15 0 0" rpy="0 1.5707963267948966 0"/>
+      <geometry>
+        <cylinder radius="0.005" length="0.3"/>
+      </geometry>
+      <material name="akshit">
+        <color rgba="1 1 1 1" />
+      </material>
+    </visual>
+    <collision>
+      <origin xyz="0.15 0 0" rpy="0 1.5707963267948966 0"/>
+      <geometry>
+        <cylinder radius="0.005" length="0.3"/>
+      </geometry>
+      <material name="akshit">
+        <color rgba="1 1 1 1" />
+      </material>
+    </collision>
+    <inertial>
+      <mass value="0.05" />
+      <origin xyz="0.15 0 0" rpy="0.0 0.0 0.0"/>
+      <inertia ixx="0.0000000001" ixy="0.0" ixz="0.0" iyy="0.0000000001" iyz="0.0" izz="0.0000000001" />
+    </inertial>
+  </link>
+  <!-- Vertical Rod Link (Height increased by 1.5x from 0.35 to 0.525) -->
+  <link name="camera_rod">
+    <visual>
+      <origin xyz="0 0 0.2625" rpy="0 0 0"/>
+      <geometry>
+        <cylinder radius="0.005" length="0.525"/>
+      </geometry>
+      <material name="akshit">
+        <color rgba="1 1 1 1" />
+      </material>
+    </visual>
+    <collision>
+      <origin xyz="0 0 0.2625" rpy="0 0 0"/>
+      <geometry>
+        <cylinder radius="0.005" length="0.525"/>
+      </geometry>
+      <material name="akshit">
+        <color rgba="1 1 1 1" />
+      </material>
+    </collision>
+    <inertial>
+      <mass value="0.1" />
+      <origin xyz="0 0 0.2625" rpy="0.0 0.0 0.0"/>
+      <inertia ixx="0.0000000001" ixy="0.0" ixz="0.0" iyy="0.0000000001" iyz="0.0" izz="0.0000000001" />
+    </inertial>
+  </link>
+  <!-- Joints -->
+  <joint name="camera_rod_joint" type="fixed">
+      <origin xyz="0.45 -0.3 0.0" rpy="0.0 0.0 1.57"/>
+      <parent link="${prefix}base_link"/>
+      <child link="camera_rod"/>
+  </joint>
+  <!-- Connect horizontal rod at the top of the vertical rod -->
+  <joint name="vertical_to_horizontal_rod" type="fixed">
+    <parent link="camera_rod"/>
+    <child link="camera_horizontal_rod"/>
+    <origin xyz="0 0 0.525" rpy="0 0 0"/>
+  </joint>
+  <!-- Connect camera to the end of the horizontal rod facing downwards -->
+  <joint name="rod_to_camera" type="fixed">
+    <parent link="camera_horizontal_rod"/>
+    <child link="camera_link"/>
+    <!-- <origin xyz="0.3 0 0" rpy="0 1.5707963267948966 0"/> -->
+    <origin xyz="0.3 0 0" rpy="0 1.5707963267948966 1.5707963267948966"/>
+  </joint>
+  <link name="camera_optical_link">
+      <inertial>
+      <mass value="0.0000000001" />
+      <origin xyz="0 0 0" rpy="0.0 0.0 0.0"/>
+      <inertia ixx="0.0000000001" ixy="0.0" ixz="0.0" iyy="0.0000000001" iyz="0.0" izz="0.0000000001" />
+    </inertial>
+  </link>
+  <joint name="optical_joint" type="fixed">
+    <parent link="camera_link"/>
+    <child link="camera_optical_link"/>
+    <origin xyz="0 0 0" rpy="-1.5707963267948966 0 -1.5707963267948966"/>
+  </joint>
+  <gazebo reference="camera_link">
+    <sensor name="rgbd_camera" type="rgbd_camera">
+      <pose>0 0 0 0 0 0</pose>
+      <camera>
+        <horizontal_fov>1.477</horizontal_fov>
+        <image>
+          <width>640</width>
+          <height>480</height>
+        </image>
+        <clip>
+          <near>0.05</near>
+          <far>10</far>
+        </clip>
+      </camera>
+      <always_on>1</always_on>
+      <update_rate>5</update_rate>
+      <visualize>true</visualize>
+      <topic>rgbd_camera</topic>
+      <gz_frame_id>camera_optical_link</gz_frame_id>
+    </sensor>
+  </gazebo>
   </xacro:macro>
 </robot>

File: rcup_assembly/src/piper_moveit_config/config/piper.srdf.xacro (robot description, xacro)
@@ -71,4 +71,6 @@
     <disable_collisions link1="link_4" link2="right_finger" reason="Never"/>
     <disable_collisions link1="link_5" link2="right_finger" reason="Never"/>
+    <disable_collisions link1="camera_link" link2="camera_horizontal_rod" reason="Adjacent"/>
+    <disable_collisions link1="camera_horizontal_rod" link2="camera_rod" reason="Adjacent"/>
     <!-- <disable_collisions link1="ax_left_finger" link2="ax_right_finger" reason="Default"/>
     <disable_collisions link1="ax_grip_base" link2="ax_right_finger" reason="Default" />

Commit message: Akshit ko dena hai

File: rcup_assembly/src/piper_description/urdf/piper_arm_macro.xacro (robot description, xacro)
@@ -253,7 +253,7 @@
   <link name="camera_rod">
     <visual>
-      <origin xyz="0 0 0.2625" rpy="0 0 0"/>
-      <geometry>
-        <cylinder radius="0.005" length="0.525"/>
+      <origin xyz="0 0 0.24" rpy="0 0 0"/>
+      <geometry>
+        <cylinder radius="0.005" length="0.48"/>
       </geometry>
       <material name="akshit">
@@ -262,7 +262,7 @@
     </visual>
     <collision>
-      <origin xyz="0 0 0.2625" rpy="0 0 0"/>
-      <geometry>
-        <cylinder radius="0.005" length="0.525"/>
+      <origin xyz="0 0 0.24" rpy="0 0 0"/>
+      <geometry>
+        <cylinder radius="0.005" length="0.48"/>
       </geometry>
       <material name="akshit">
@@ -286,5 +286,5 @@
     <parent link="camera_rod"/>
     <child link="camera_horizontal_rod"/>
-    <origin xyz="0 0 0.525" rpy="0 0 0"/>
+    <origin xyz="0 0 0.48" rpy="0 0 0"/>
   </joint>
   <!-- Connect camera to the end of the horizontal rod facing downwards -->
