Commit message: Lessgooo all donee

File: rcup_final/src/piper_moveit_config/config/piper.srdf.xacro (robot description, xacro)
@@ -36,6 +36,6 @@
     </group_state>
     <group_state name="closed" group="gripper">
-        <joint name="gripper_joint" value="0.01"/>
-         <joint name="mimic_gripper_joint" value="0.01"/>
+        <joint name="gripper_joint" value="0.012"/>
+         <joint name="mimic_gripper_joint" value="0.012"/>
     </group_state>
     <!-- <group_state name="open" group="clamper">
